File: Circuit/PreFinal/EEG.sch (EAGLE design)
At the start: 100 parts

Commit message: board development
Changed lines of the file:
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@@
 <wire x1="-89" y1="-27.3" x2="-89.08" y2="-27.3" width="0.1524" layer="91"/>
 <pinref part="B_RES_5" gate="G$1" pin="1"/>
-<wire x1="-89.08" y1="-27.3" x2="-86.32" y2="-27.3" width="0.1524" layer="91"/>
 <junction x="-89.08" y="-27.3"/>
 <pinref part="B_RES_6" gate="G$1" pin="2"/>
 <wire x1="-89.18" y1="-22.2" x2="-89" y2="-16.3" width="0.1524" layer="91"/>
 <wire x1="-89" y1="-16.3" x2="-89.08" y2="-16.3" width="0.1524" layer="91"/>
+<wire x1="-89.08" y1="-16.3" x2="-89.08" y2="-27.3" width="0.1524" layer="91"/>
+<wire x1="-89.08" y1="-27.3" x2="-86.32" y2="-27.3" width="0.1524" layer="91"/>
+<junction x="-89.08" y="-16.3"/>
 </segment>
 </net>
