File: Circuit/PreFinal/EEG.brd (EAGLE design)
At the start: 160 x 100 mm, 100 parts

Commit message: board development
Parts:
- moved R10 96.2 mm to (101.3, 66.8), flipped to the bottom, turned to 270 degrees
- moved U$24 88.8 mm to (97.2, 66.0), flipped to the bottom
- moved U$54 80.4 mm to (92.5, 65.8), flipped to the bottom, turned to 90 degrees
- moved U$55 78.7 mm to (90.2, 66.6), flipped to the bottom, turned to 270 degrees
- moved R9 78.3 mm to (91.3, 66.6), flipped to the bottom
- moved U$33 68.5 mm to (61.7, 62.5), turned to 90 degrees
- moved B_RES_3 67.6 mm to (59.3, 51.5), turned to 180 degrees
- moved C2 66.7 mm to (96.7, 75.7), flipped to the bottom, turned to 90 degrees
- moved R5 66.7 mm to (94.7, 75.2), flipped to the bottom, turned to 90 degrees
- moved R8 66.1 mm to (96.7, 73.6), flipped to the bottom
- moved B_RES_1 66.1 mm to (60.8, 51.9)
- moved B_CAP_1 65.6 mm to (59.3, 52.4)
- moved BUTTON2 64.9 mm to (53.2, 51.5), turned to 0 degrees
- moved B_RES_2 64.9 mm to (59.3, 53.3), turned to 0 degrees
- moved BOOT1 64.7 mm to (59.0, 60.7), turned to 270 degrees
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Connections:
- net GND: now also U$22.P$1, U$22.P$2, U$22.P$3, U$22.P$4
Routing:
- net V+: track 0.00 -> 132.5 mm, vias 0 -> 9
- net GND: track 0.00 -> 36.7 mm
- net N$21: track 0.00 -> 18.0 mm, vias 0 -> 1
- net N$3: track 0.00 -> 17.5 mm, vias 0 -> 1
- net N$5: track 0.00 -> 14.2 mm, vias 0 -> 1
- net N$20: track 0.00 -> 10.9 mm
- net N$4: track 0.00 -> 10.8 mm
- net N$19: track 0.00 -> 10.8 mm
- net VDD: track 0.00 -> 10.4 mm
- net N$25: track 0.00 -> 9.60 mm
- net N$27: track 0.00 -> 9.21 mm
- net N$26: track 0.00 -> 8.55 mm
- net N$16: track 0.00 -> 8.18 mm
- net N$14: track 0.00 -> 7.05 mm
- net N$13: track 0.00 -> 7.03 mm
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Other:
- outline, holes or cut-outs redrawn

Commit message: Add app prototype
Parts:
- moved R10 48.1 mm to (53.2, 69.2), turned to 0 degrees
- moved U$24 45.3 mm to (52.5, 72.9), turned to 90 degrees
- moved U$15 43.0 mm to (71.6, 60.9), turned to 90 degrees
- moved U$11 42.4 mm to (70.8, 60.9), turned to 90 degrees
- moved U$54 42.1 mm to (51.9, 77.2), turned to 180 degrees
- moved U$9 41.7 mm to (71.2, 59.0), turned to 0 degrees
- moved RG 39.6 mm to (80.3, 57.3)
- moved U$27 38.8 mm to (70.6, 62.9), turned to 0 degrees
- moved U$4 38.4 mm to (76.5, 57.3), turned to 0 degrees
- moved R9 38.0 mm to (54.8, 76.8), turned to 270 degrees
- moved U$12 36.5 mm to (60.0, 57.4)
- moved U$20 36.5 mm to (60.0, 58.3)
- moved U$55 35.9 mm to (55.8, 76.8), turned to 90 degrees
- moved U$16 35.6 mm to (66.5, 58.3)
- moved U$17 35.2 mm to (63.3, 54.1), turned to 180 degrees
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Routing:
- net V-: track 0.00 -> 50.7 mm, vias 0 -> 3
- net V+: track 132.5 -> 179.2 mm, vias 9 -> 11
- net N$48: track 4.72 -> 44.9 mm, vias 0 -> 2
- net VDD: track 10.4 -> 49.3 mm, vias 0 -> 1
- net N$68: track 0.00 -> 33.4 mm, vias 0 -> 2
- net GND: track 36.7 -> 68.4 mm, vias 0 -> 5
- net N$23: track 6.55 -> 32.4 mm
- net N$57: track 0.00 -> 25.4 mm
- net N$46: track 4.07 -> 26.0 mm
- net N$62: track 0.00 -> 13.1 mm
- net N$63: track 1.40 -> 14.0 mm
- net N$60: track 0.00 -> 9.47 mm
- net N$21: track 18.0 -> 26.7 mm
- net N$44: track 4.43 -> 11.3 mm
- net N$58: track 0.00 -> 6.65 mm
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- added copper zone on layer 16, net GND

Commit message: update data
Other:
- board size 160 x 100 mm -> 32.8 x 38.1 mm
